Commit message: added camera frames

File: fetch_description/robots/stand_alone_arm.urdf (robot description, URDF)
Before this commit: robot stand_alone_arm, 16 links, 15 joints
Links:
- added link camera_depth_frame
- added link camera_depth_optical_frame
- added link camera_rgb_frame
- added link camera_rgb_optical_frame
Joints:
- added joint camera_depth_joint: type fixed, parent camera_link, child camera_depth_frame, origin xyz=0 -0.0093 0 rpy=0 0 0
- added joint camera_depth_optical_joint: type fixed, parent camera_link, child camera_depth_optical_frame, origin xyz=0 -0.0093 0 rpy=0 0 0
- added joint camera_rgb_joint: type fixed, parent camera_link, child camera_rgb_frame, origin xyz=0 -0.0093 0 rpy=0 0 0
- added joint camera_rgb_optical_joint: type fixed, parent camera_link, child camera_rgb_optical_frame, origin xyz=0 -0.0093 0 rpy=0 0 0
- joint camera_joint: origin xyz=0 1.5383 1.074 rpy=0 0 0 -> xyz=0 1.5233 1.049 rpy=0 0 0

Commit message: changed URDF and paths

File: fetch_description/robots/stand_alone_arm.urdf (robot description, URDF)
Before this commit: robot stand_alone_arm, 20 links, 19 joints
Joints:
- joint forearm_roll_joint: type revolute -> continuous
